File: PCB/ATOM.kicad_pcb (KiCad board)
At the start: 2 copper layers, 284.9 x 112.7 mm, 0 parts

Commit message: route matrix
Parts:
- added D1: BAV70, ATOM:SOT-23, F.Cu at (101.5, 119.3)
- added D10: BAV70, ATOM:SOT-23, F.Cu at (244.2, 150.5)
- added D11: BAV70, ATOM:SOT-23, F.Cu at (279.2, 133.8)
- added D12: BAV70, ATOM:SOT-23, F.Cu at (319.1, 135.5)
- added D13: BAV70, ATOM:SOT-23, F.Cu at (90.5, 156.8)
- added D14: BAV70, ATOM:SOT-23, F.Cu at (130.9, 156.8)
- added D15: BAV70, ATOM:SOT-23, F.Cu at (167.7, 166.6)
- added D16: BAV70, ATOM:SOT-23, F.Cu at (249.2, 168.9)
- added D17: BAV70, ATOM:SOT-23, F.Cu at (284.1, 152.2)
- added D18: BAV70, ATOM:SOT-23, F.Cu at (324.0, 153.7)
- added D19: BAV70, ATOM:SOT-23, F.Cu at (162.8, 185.0)
- added D2: BAV70, ATOM:SOT-23, F.Cu at (140.8, 120.0)
- added D20: BAV70, ATOM:SOT-23, F.Cu at (208.1, 199.5)
- added D21: BAV70, ATOM:SOT-23, F.Cu at (254.1, 187.4)
- added D3: BAV70, ATOM:SOT-23, F.Cu at (177.6, 129.8)
- added D4: BAV70, ATOM:SOT-23, F.Cu at (239.3, 132.1)
- added D5: BAV70, ATOM:SOT-23, F.Cu at (274.3, 115.4)
- added D6: BAV70, ATOM:SOT-23, F.Cu at (314.1, 116.9)
- added D7: BAV70, ATOM:SOT-23, F.Cu at (96.6, 137.7)
- added D8: BAV70, ATOM:SOT-23, F.Cu at (135.8, 138.5)
- added D9: BAV70, ATOM:SOT-23, F.Cu at (172.6, 148.4)
- added SW1: SW_Push, ATOM:SW_Hotswap_Kailh_CPG1353, F.Cu at (87.3, 108.3)
- added SW10: SW_Push, ATOM:SW_Hotswap_Kailh_CPG1353, F.Cu at (276.1, 112.6)
- added SW11: SW_Push, ATOM:SW_Hotswap_Kailh_CPG1353, F.Cu at (296.4, 114.4)
- added SW12: SW_Push, ATOM:SW_Hotswap_Kailh_CPG1353, F.Cu at (315.4, 111.9)
- added SW13: SW_Push, ATOM:SW_Hotswap_Kailh_CPG1353, F.Cu at (82.4, 126.7)
- added SW14: SW_Push, ATOM:SW_Hotswap_Kailh_CPG1353, F.Cu at (101.4, 129.2)
- added SW15: SW_Push, ATOM:SW_Hotswap_Kailh_CPG1353, F.Cu at (121.7, 127.3)
- added SW16: SW_Push, ATOM:SW_Hotswap_Kailh_CPG1353, F.Cu at (141.3, 127.7)
- added SW17: SW_Push, ATOM:SW_Hotswap_Kailh_CPG1353, F.Cu at (158.5, 137.2)
- added SW18: SW_Push, ATOM:SW_Hotswap_Kailh_CPG1353, F.Cu at (176.3, 144.3)
- added SW19: SW_Push, ATOM:SW_Hotswap_Kailh_CPG1353, F.Cu at (226.5, 148.0)
- added SW2: SW_Push, ATOM:SW_Hotswap_Kailh_CPG1353, F.Cu at (106.4, 110.8)
- added SW20: SW_Push, ATOM:SW_Hotswap_Kailh_CPG1353, F.Cu at (244.3, 140.8)
- added SW21: SW_Push, ATOM:SW_Hotswap_Kailh_CPG1353, F.Cu at (261.4, 131.3)
- added SW22: SW_Push, ATOM:SW_Hotswap_Kailh_CPG1353, F.Cu at (281.1, 131.0)
- added SW23: SW_Push, ATOM:SW_Hotswap_Kailh_CPG1353, F.Cu at (301.3, 132.8)
- added SW24: SW_Push, ATOM:SW_Hotswap_Kailh_CPG1353, F.Cu at (320.3, 130.3)
- added SW25: SW_Push, ATOM:SW_Hotswap_Kailh_CPG1353, F.Cu at (77.5, 145.1)
- added SW26: SW_Push, ATOM:SW_Hotswap_Kailh_CPG1353, F.Cu at (96.5, 147.6)
- added SW27: SW_Push, ATOM:SW_Hotswap_Kailh_CPG1353, F.Cu at (116.7, 145.7)
- added SW28: SW_Push, ATOM:SW_Hotswap_Kailh_CPG1353, F.Cu at (136.4, 146.1)
- added SW29: SW_Push, ATOM:SW_Hotswap_Kailh_CPG1353, F.Cu at (153.5, 155.6)
- added SW3: SW_Push, ATOM:SW_Hotswap_Kailh_CPG1353, F.Cu at (126.6, 108.9)
- added SW30: SW_Push, ATOM:SW_Hotswap_Kailh_CPG1353, F.Cu at (171.4, 162.7)
- added SW31: SW_Push, ATOM:SW_Hotswap_Kailh_CPG1353, F.Cu at (231.4, 166.4)
- added SW32: SW_Push, ATOM:SW_Hotswap_Kailh_CPG1353, F.Cu at (249.2, 159.2)
- added SW33: SW_Push, ATOM:SW_Hotswap_Kailh_CPG1353, F.Cu at (266.4, 149.7)
- added SW34: SW_Push, ATOM:SW_Hotswap_Kailh_CPG1353, F.Cu at (286.0, 149.4)
- added SW35: SW_Push, ATOM:SW_Hotswap_Kailh_CPG1353, F.Cu at (306.2, 151.2)
- added SW36: SW_Push, ATOM:SW_Hotswap_Kailh_CPG1353, F.Cu at (325.3, 148.7)
- added SW37: SW_Push, ATOM:SW_Hotswap_Kailh_CPG1353, F.Cu at (148.6, 174.0)
- added SW38: SW_Push, ATOM:SW_Hotswap_Kailh_CPG1353, F.Cu at (166.4, 181.1)
- added SW39: SW_Push, ATOM:SW_Hotswap_Kailh_CPG1353, F.Cu at (184.2, 188.5)
- added SW4: SW_Push, ATOM:SW_Hotswap_Kailh_CPG1353, F.Cu at (146.2, 109.3)
- added SW40: SW_Push, ATOM:SW_Hotswap_Kailh_CPG1353, F.Cu at (218.6, 192.1)
- added SW41: SW_Push, ATOM:SW_Hotswap_Kailh_CPG1353, F.Cu at (236.3, 184.8)
- added SW42: SW_Push, ATOM:SW_Hotswap_Kailh_CPG1353, F.Cu at (254.1, 177.6)
- added SW5: SW_Push, ATOM:SW_Hotswap_Kailh_CPG1353, F.Cu at (163.4, 118.8)
- added SW6: SW_Push, ATOM:SW_Hotswap_Kailh_CPG1353, F.Cu at (181.2, 125.9)
- added SW7: SW_Push, ATOM:SW_Hotswap_Kailh_CPG1353, F.Cu at (221.5, 129.6)
- added SW8: SW_Push, ATOM:SW_Hotswap_Kailh_CPG1353, F.Cu at (239.3, 122.4)
- added SW9: SW_Push, ATOM:SW_Hotswap_Kailh_CPG1353, F.Cu at (256.5, 112.9)
Routing:
- net ROW2: track 0.00 -> 257.0 mm, vias 0 -> 6
- net ROW1: track 0.00 -> 246.6 mm, vias 0 -> 6
- net ROW0: track 0.00 -> 234.4 mm, vias 0 -> 6
- net ROW3: track 0.00 -> 104.3 mm, vias 0 -> 3
- net COL4: track 0.00 -> 83.8 mm
- net COL7: track 0.00 -> 79.9 mm
- net COL8: track 0.00 -> 67.9 mm
- net COL6: track 0.00 -> 65.9 mm
- net COL3: track 0.00 -> 64.1 mm
- net COL5: track 0.00 -> 62.1 mm
- net COL0: track 0.00 -> 42.5 mm
- net COL9: track 0.00 -> 40.9 mm
- net COL2: track 0.00 -> 40.9 mm
- net COL1: track 0.00 -> 40.9 mm
- net COL10: track 0.00 -> 40.9 mm
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Other:
- board size 284.9 x 112.7 mm -> 280.4 x 109.5 mm

Commit message: route daughterboard
Parts:
- added ?: , , F.Cu at (317.7, 167.7)
- added ?: , , F.Cu at (321.2, 180.7)
- added C1: 100nF, ATOM:C_0603_1608Metric_Pad1.08x0.95mm_HandSolder, F.Cu at (315.4, 169.7)
- added F1: 500mA, ATOM:Fuse_1206_3216Metric_Pad1.42x1.75mm_HandSolder, F.Cu at (321.2, 167.0)
- added J1: USB_C_Receptacle_USB2.0_16P, ATOM:USB_C_Receptacle_HRO_TYPE-C-31-M-12, F.Cu at (323.5, 173.1)
- added J2: Conn_01x03, ATOM:JST_PH_S3B-PH-SM4-TB_1x03-1MP_P2.00mm_Horizontal, F.Cu at (310.2, 176.7)
- added R1: 5.1K, ATOM:R_0603_1608Metric_Pad0.98x0.95mm_HandSolder, F.Cu at (317.7, 178.4)
- added R2: 5.1K, ATOM:R_0603_1608Metric_Pad0.98x0.95mm_HandSolder, F.Cu at (315.8, 171.1)
- added R3: 1M, ATOM:R_0603_1608Metric_Pad0.98x0.95mm_HandSolder, F.Cu at (318.1, 179.9)
- added REF**: MountingHole_2.2mm_M2, ATOM:MountingHole_2.2mm_M2, F.Cu at (324.7, 165.8)
- added REF**: MountingHole_2.2mm_M2, ATOM:MountingHole_2.2mm_M2, F.Cu at (328.2, 178.8)
- added U1: E73-2G4M08S1C-52840, ATOM:E73-2G4M08S1C-52840, F.Cu at (212.4, 228.4)
- added U2: USBLC6-2SC6, ATOM:TSOT-23-6_HandSoldering, F.Cu at (316.7, 174.9)
Routing:
- net Net-(F1-Pad1): track 0.00 -> 13.3 mm
- net USB-: track 0.00 -> 8.31 mm
- net GND: track 0.00 -> 6.64 mm, vias 0 -> 1
- net DATA-: track 0.00 -> 6.16 mm
- net DATA+: track 0.00 -> 5.62 mm
- net USB+: track 0.00 -> 5.58 mm
- net VBUS: track 0.00 -> 5.33 mm
- net Net-(J1-CC1): track 0.00 -> 3.83 mm
- net Net-(J1-CC2): track 0.00 -> 3.54 mm
- added copper zone on B.Cu, net GND
- added copper zone on F.Cu, net GND
Other:
- outline, holes or cut-outs redrawn
